Commit message: 3finger_gripper_mod_1

File: iiwa_tool/iiwa_tool_description/urdf/iiwa14_3finger_gripper.urdf.xacro (robot description, xacro)
@@ -8,5 +8,5 @@
   <!--  Arguments for the iiwa14 macro  -->
   <xacro:arg name="hardware_interface" default="PositionJointInterface"/>
-  <xacro:arg name="robot_name" default="iiwa14"/>
+  <xacro:arg name="robot_name" default="iiwa"/>
   <!--  Define the origin of your 3D space
   Here we define a box lying at 0,0,0 with some dimensions, in reality our robot is place on top of a metal cart with those dimensions.
@@ -17,13 +17,13 @@
   <link name="world">
     <visual>
-      <origin xyz="0 0 0.42" rpy="0 0 0"/>
+      <origin xyz="0 0 1.5" rpy="0 0 0"/>
       <geometry>
-	<box size="0.68 0.605 0.84"/>
+	<box size="1 2 3"/>
       </geometry>
     </visual>
     <collision>
-      <origin xyz="0 0 0.42" rpy="0 0 0"/>
+      <origin xyz="0 0 1.5" rpy="0 0 0"/>
       <geometry>
-	<box size="0.68 0.605 0.84"/>
+	<box size="1 2 3"/>
       </geometry>
     </collision>
@@ -34,8 +34,8 @@
   <!-- Here we insert an iiwa14 robot in the scene, it's origin is just on top of the box previously defined. You can use 0,0,0 if you don't have that. -->
   <xacro:iiwa14 hardware_interface="$(arg hardware_interface)" robot_name="$(arg robot_name)" parent="world">
-    <origin xyz="0 0 0.84" rpy="0 0 0"/>
+    <origin xyz="0 0 3" rpy="0 0 0"/>
   </xacro:iiwa14>
   <!-- Tool properties -->
-  <property name="tool_mass" value="0.200" />
+  <property name="tool_mass" value="3.200" />
   <property name="tool_joint_offset" value="0.00 0.00 0.00" />
   <property name="tool_link_offset" value="0.00 0.00 0.1275" />
@@ -43,5 +43,5 @@
   There is no offset between the two, that means the tool is attached at the robot flange. -->
   <joint name="tool_joint" type="fixed">
-    <parent link="iiwa_link_ee" />
+    <parent link="$(arg robot_name)_link_ee" />
     <child link = "tool_link" />
     <origin xyz="${tool_joint_offset}" rpy="0 ${PI/2.0} 0" />

Commit message: robot base box dimension

File: iiwa_tool/iiwa_tool_description/urdf/iiwa14_3finger_gripper.urdf.xacro (robot description, xacro)
@@ -17,13 +17,13 @@
   <link name="world">
     <visual>
-      <origin xyz="0 0 1.5" rpy="0 0 0"/>
+      <origin xyz="0 0 0.38" rpy="0 0 0"/>
       <geometry>
-	<box size="1 2 3"/>
+	<box size="0.60 0.60 0.76"/>
       </geometry>
     </visual>
     <collision>
-      <origin xyz="0 0 1.5" rpy="0 0 0"/>
+      <origin xyz="0 0 0.38" rpy="0 0 0"/>
       <geometry>
-	<box size="1 2 3"/>
+	<box size="0.60 0.60 0.76"/>
       </geometry>
     </collision>
@@ -34,5 +34,5 @@
   <!-- Here we insert an iiwa14 robot in the scene, it's origin is just on top of the box previously defined. You can use 0,0,0 if you don't have that. -->
   <xacro:iiwa14 hardware_interface="$(arg hardware_interface)" robot_name="$(arg robot_name)" parent="world">
-    <origin xyz="0 0 3" rpy="0 0 0"/>
+    <origin xyz="0 0 0.76" rpy="0 0 0"/>
   </xacro:iiwa14>
   <!-- Tool properties -->

Commit message: xacro of 3finger_gripper

File: iiwa_tool/iiwa_tool_description/urdf/iiwa14_3finger_gripper.urdf.xacro (robot description, xacro)
@@ -6,4 +6,634 @@
   <!--Import the iiwa14 macro -->
   <xacro:include filename="$(find iiwa_description)/urdf/iiwa14.xacro"/>
+  <!--Build finger model -->
+  <xacro:macro name="robotiq_finger" params="prefix">
+    <!-- Link list -->
+    <!-- Link 0 -->
+    <link name="${prefix}link_0">
+      <visual>
+        <origin xyz="0 0 0" rpy="0 0 0"/>
+        <geometry>
+          <mesh filename="package://robotiq_hand_description/meshes/s-model_articulated/visual/link_0.STL" />
+        </geometry>
+        <material name="green">
+          <color rgba="0 1 0 1"/>
+        </material>
+      </visual>
+      <collision>
+        <origin rpy="0 0 0" xyz="0 0 0"/>
+        <geometry>
+          <mesh filename="package://robotiq_hand_description/meshes/s-model_articulated/collision/link_0.STL" />
+        </geometry>
+        <material name="yellow">
+          <color rgba="0 1 1 1"/>
+        </material>
+      </collision>
+      <inertial>
+        <mass value="0.1"/>
+        <origin xyz="-0.01 0 0"/>
+        <inertia ixx="0.000018" ixy="0" ixz="0" iyy="0.000025" iyz="0" izz="0.000025"/>
+      </inertial>
+    </link>
+    <gazebo reference="${prefix}link_0">
+      <mu1>1.1</mu1>
+      <mu2>1.1</mu2>
+    </gazebo>
+    <!-- Link 1 -->
+    <link name="${prefix}link_1">
+      <visual>
+        <origin rpy="0 0 ${3.1416/2}" xyz="0 0.05717 0"/>
+        <geometry>
+          <mesh filename="package://robotiq_hand_description/meshes/s-model_articulated/visual/link_1.STL" />
+        </geometry>
+        <material name="green"/>
+      </visual>
+      <collision>
+        <origin rpy="0 0 ${3.1416/2}" xyz="0 0.05717 0"/>
+        <geometry>
+          <mesh filename="package://robotiq_hand_description/meshes/s-model_articulated/collision/link_1.STL"/>
+        </geometry>
+        <material name="yellow">
+          <color rgba="0 1 1 1"/>
+        </material>
+      </collision>
+      <inertial>
+        <origin rpy="0 0 ${3.1416/2}" xyz="0.00053 0.03218 0"/>
+        <mass value="0.047"/>
+        <inertia ixx= "0.00000499332"
+                 ixy= "0.00000091312"
+                 ixz="-0.00000000120"
+                 iyy= "0.00006434531"
+                 iyz="-0.00000000007"
+                 izz= "0.00006061917"/>
+      </inertial>
+    </link>
+    <gazebo reference="${prefix}link_1">
+      <mu1>1.1</mu1>
+      <mu2>1.1</mu2>
+      <minDepth>0.001</minDepth>
+    </gazebo>
+    <!-- Link 2 -->
+    <link name="${prefix}link_2">
+      <visual>
+        <origin rpy="0 0 ${3.1416/2}" xyz="0 0.03810 0.0075"/>
+        <geometry>
+          <mesh filename="package://robotiq_hand_description/meshes/s-model_articulated/visual/link_2.STL" />
+        </geometry>
+        <material name="green"/>
+      </visual>
+      <collision>
+        <origin rpy="0 0 ${3.1416/2}" xyz="0 0.03810 0.0075"/>
+          <geometry>
+            <mesh filename="package://robotiq_hand_description/meshes/s-model_articulated/collision/link_2.STL"/>
+          </geometry>
+        <material name="yellow"/>
+      </collision>
+      <inertial>
+        <origin rpy="0 0 ${3.1416/2}" xyz="0.00048 0.02167 0.00018"/>
+        <mass value="0.03284"/>
+        <inertia ixx="0.00000348008"
+                 ixy="0.00000031940"
+                 ixz="0.00000013041"
+                 iyy="0.00002248123"
+                 iyz="0.00000000291"
+                 izz="0.00001986346"/>
+      </inertial>
+    </link>
+    <gazebo reference="${prefix}link_2">
+      <mu1>1.1</mu1>
+      <mu2>1.1</mu2>
+      <minDepth>0.001</minDepth>
+    </gazebo>
+    <!-- Link 3 -->
+    <link name="${prefix}link_3">
+      <visual>
+        <origin xyz="0 0 0" rpy="0 0 0"/>
+        <geometry>
+          <mesh filename="package://robotiq_hand_description/meshes/s-model_articulated/visual/link_3.STL" />
+        </geometry>
+        <material name="green"/>
+      </visual>
+      <collision>
+        <origin xyz="0 0 0" rpy="0 0 0"/>
+        <geometry>
+          <mesh filename="package://robotiq_hand_description/meshes/s-model_articulated/collision/link_3.STL"/>
+        </geometry>
+        <material name="yellow"/>
+      </collision>
+      <inertial>
+        <origin rpy="0 0 0" xyz="0.01626 0.00049 0.0002"/>
+        <mass value="0.03354"/>
+        <inertia ixx="0.00000305151"
+                 ixy="0.00000089792"
+                 ixz="0.00000000249"
+                 iyy="0.00001427978"
+                 iyz="-0.00000001191"
+                 izz="0.00001264126"/>
+      </inertial>
+    </link>
+    <gazebo reference="${prefix}link_3">
+      <mu1>1.1</mu1>
+      <mu2>1.1</mu2>
+      <minDepth>0.001</minDepth>
+    </gazebo>
+    <!-- Link proximal actuating hinge -->
+    <link name="${prefix}link_proximal_actuating_hinge">
+      <visual>
+        <origin rpy="0 0 0" xyz="0.01429 0 0"/>
+        <geometry>
+          <box size="0.02858 .0075 .002"/>
+        </geometry>
+      </visual>
+      <collision>
+        <origin rpy="0 0 0" xyz="0.01429 0 0"/>
+         <geometry>
+          <box size="0.02858 .0075 .002"/>
+        </geometry>
+      </collision>
+      <inertial>
+        <origin rpy="0 0 0" xyz="0.0012 -0.00162 -0.00161"/>
+        <mass value="0.02647"/>
+        <inertia ixx= "0.00000156447"
+                 ixy= "0.000000236226"
+                 ixz="-0.00000014862"
+                 iyy= "0.00000221068"
+                 iyz="-0.00000014369"
+                 izz= "0.00000323175"/>
+      </inertial>
+    </link>
+    <gazebo reference="${prefix}link_proximal_actuating_hinge">
+      <mu1>1.1</mu1>
+      <mu2>1.1</mu2>
+    </gazebo>
+    <!-- Link paraproximal actuating hinge -->
+    <link name="${prefix}link_paraproximal_actuating_hinge">
+      <visual>
+        <origin rpy="0 0 0" xyz="0.01143 0 0"/>
+        <geometry>
+          <box size="0.02286 .0075 .002"/>
+        </geometry>
+      </visual>
+      <collision>
+        <origin rpy="0 0 0" xyz="0.01143 0 0"/>
+         <geometry>
+          <box size="0.02286 .0075 .002"/>
+        </geometry>
+      </collision>
+      <inertial>
+        <origin rpy="0 0 0" xyz="0.0064 0 0"/>
+        <!-- copied from proximal_actuating_hinge -->
+        <mass value="0.00362"/>
+        <inertia ixx= "0.00000012043"
+                 ixy= "0"
+                 ixz= "0"
+                 iyy= "0.00000053588"
+                 iyz= "0"
+                 izz= "0.00000065322"/>
+      </inertial>
+    </link>
+    <gazebo reference="${prefix}link_paraproximal_actuating_hinge">
+      <mu1>1.1</mu1>
+      <mu2>1.1</mu2>
+    </gazebo>
+    <!-- Link proximal actuating bar -->
+    <link name="${prefix}link_proximal_actuating_bar">
+      <visual>
+        <origin rpy="0 0 0" xyz="0.026789 0 0"/>
+        <geometry>
+          <box size="0.05398 .0075 .002"/>
+        </geometry>
+      </visual>
+      <collision>
+        <origin rpy="0 0 0" xyz="0.026789 0 0"/>
+         <geometry>
+          <box size="0.05398 .0075 .002"/>
+        </geometry>
+      </collision>
+      <inertial>
+        <origin rpy="0 0 0" xyz="0.02699 -0.00122 0"/>
+        <mass value="0.00659"/>
+        <inertia ixx= "0.00000008348"
+                 ixy="-0.0000002179"
+                 ixz= "0.00000000134"
+                 iyy= "0.00000719076"
+                 iyz= "0"
+                 izz= "0.00000718272"/>
+      </inertial>
+    </link>
+    <gazebo reference="${prefix}link_proximal_actuating_bar">
+      <mu1>1.1</mu1>
+      <mu2>1.1</mu2>
+    </gazebo>
+    <!-- Link paraproximal bar -->
+    <link name="${prefix}link_paraproximal_bar">
+      <visual>
+        <origin rpy="0 0 0" xyz="0.02885 0 0"/>
+        <geometry>
+          <box size="0.05770 .0075 .002"/>
+        </geometry>
+      </visual>
+      <collision>
+        <origin rpy="0 0 0" xyz="0.02885 0 0"/>
+         <geometry>
+          <box size="0.05770 .0075 .002"/>
+        </geometry>
+      </collision>
+      <inertial>
+        <origin rpy="0 0 0" xyz="0.02858 -0.00129 0"/>
+        <mass value="0.00732"/>
+        <inertia ixx= "0.00000009065"
+                 ixy="-0.00000027047"
+                 ixz= "0.00000000142"
+                 iyy= "0.00000878034"
+                 iyz= "0"
+                 izz= "0.00000877558"/>
+      </inertial>
+    </link>
+    <gazebo reference="${prefix}link_paraproximal_bar">
+      <mu1>1.1</mu1>
+      <mu2>1.1</mu2>
+    </gazebo>
+    <!-- Link median actuating hinge -->
+    <link name="${prefix}link_median_actuating_hinge">
+      <visual>
+        <origin rpy="0 0 0" xyz="0 0 0"/>
+        <geometry>
+          <box size=".02 .02 .002"/>
+        </geometry>
+      </visual>
+      <collision>
+        <origin rpy="0 0 0" xyz="0 0 0"/>
+         <geometry>
+          <box size=".02 .02 .002"/>
+        </geometry>
+      </collision>
+      <inertial>
+        <origin rpy="0 0 0" xyz="0.0092 0.00514 0"/>
+        <mass value="0.00359"/>
+        <inertia ixx= "0.00000024735"
+                 ixy= "0.00000023619"
+                 ixz= "0"
+                 iyy= "0.00000047681"
+                 iyz= "0"
+                 izz= "0.00000071813"/>
+      </inertial>
+    </link>
+    <gazebo reference="${prefix}link_median_actuating_hinge">
+      <mu1>1.1</mu1>
+      <mu2>1.1</mu2>
+    </gazebo>
+    <!-- Link median bar -->
+    <link name="${prefix}link_median_bar">
+      <visual>
+        <origin rpy="0 0 0" xyz="0.01905 0 0"/>
+        <geometry>
+          <box size="0.0381 .0075 .002"/>
+        </geometry>
+      </visual>
+      <collision>
+        <origin rpy="0 0 0" xyz="0.01905 0 0"/>
+         <geometry>
+          <box size="0.0381 .0075 .002"/>
+        </geometry>
+      </collision>
+      <inertial>
+        <origin rpy="0 0 0" xyz="0.01905 -0.00107 0"/>
+        <mass value="0.00538"/>
+        <inertia ixx= "0.00000006639"
+                 ixy="-0.00000010996"
+                 ixz= "0.00000000094"
+                 iyy= "0.00000305318"
+                 iyz= "0"
+                 izz= "0.00000304657"/>
+      </inertial>
+    </link>
+    <gazebo reference="${prefix}link_median_bar">
+      <mu1>1.1</mu1>
+      <mu2>1.1</mu2>
+    </gazebo>
+    <!-- Link paramedian hinge -->
+    <link name="${prefix}link_paramedian_hinge">
+      <visual>
+        <origin rpy="0 0 0" xyz="0 0 0"/>
+        <geometry>
+          <box size=".02 .02 .002"/>
+        </geometry>
+      </visual>
+      <collision>
+        <origin rpy="0 0 0" xyz="0 0 0"/>
+         <geometry>
+          <box size=".02 .02 .002"/>
+        </geometry>
+      </collision>
+      <inertial>
+        <origin rpy="0 0 0" xyz="-0.01025 0.00046 0"/>
+        <mass value="0.00276"/>
+        <inertia ixx= "0.00000004213"
+                 ixy="-0.00000001491"
+                 ixz= "0"
+                 iyy= "0.00000050258"
+                 iyz= "0"
+                 izz= "0.00000054007"/>
+      </inertial>
+    </link>
+    <gazebo reference="${prefix}link_paramedian_hinge">
+      <mu1>1.1</mu1>
+      <mu2>1.1</mu2>
+    </gazebo>
+    <!-- Link median bar underactuated -->
+    <link name="${prefix}link_median_bar_underactuated">
+      <visual>
+        <origin rpy="0 0 0" xyz="0.01905 0 0"/>
+        <geometry>
+          <box size="0.0381 .0075 .002"/>
+        </geometry>
+      </visual>
+      <collision>
+        <origin rpy="0 0 0" xyz="0.01905 0 0"/>
+         <geometry>
+          <box size="0.0381 .0075 .002"/>
+        </geometry>
+      </collision>
+      <inertial>
+        <origin rpy="0 0 0" xyz="0.01905 -0.00107 0"/>
+        <mass value="0.00538"/>
+        <inertia ixx= "0.00000006639"
+                 ixy="-0.00000010996"
+                 ixz="-0.00000000094"
+                 iyy= "0.00000305318"
+                 iyz= "0"
+                 izz= "0.00000304657"/>
+      </inertial>
+    </link>
+    <gazebo reference="${prefix}link_median_bar_underactuated">
+      <mu1>1.1</mu1>
+      <mu2>1.1</mu2>
+    </gazebo>
+    <!-- Link paradistal hinge -->
+    <link name="${prefix}link_paradistal_hinge">
+      <visual>
+        <origin rpy="0 0 0" xyz="0 0 0"/>
+        <geometry>
+          <box size=".02 .02 .002"/>
+        </geometry>
+      </visual>
+      <collision>
+        <origin rpy="0 0 0" xyz="0 0 0"/>
+         <geometry>
+          <box size=".02 0.02 .002"/>
+        </geometry>
+      </collision>
+      <inertial>
+        <origin rpy="0 0 0" xyz="0.00548 0 0"/>
+        <mass value="0.00158"/>
+        <inertia ixx= "0.00000001907"
+                 ixy= "0"
+                 ixz= "0"
+                 iyy= "0.00000010970"
+                 iyz= "0"
+                 izz= "0.00000012610"/>
+      </inertial>
+    </link>
+    <gazebo reference="${prefix}link_paradistal_hinge">
+      <mu1>1.1</mu1>
+      <mu2>1.1</mu2>
+    </gazebo>
+    <!-- End of link list -->
+    <!-- Joint list -->
+    <!-- Joint proximal actuating hinge -->
+    <joint name="${prefix}joint_proximal_actuating_hinge" type="revolute">
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
Commit message: modif for xacro of 3finger_gripper

File: iiwa_tool/iiwa_tool_description/urdf/iiwa14_3finger_gripper.urdf.xacro (robot description, xacro)
@@ -14,5 +14,5 @@
         <origin xyz="0 0 0" rpy="0 0 0"/>
         <geometry>
-          <mesh filename="package://robotiq_hand_description/meshes/s-model_articulated/visual/link_0.STL" />
+          <mesh filename="package://iiwa_tool_description/meshes/visual/link_0.STL" />
         </geometry>
         <material name="green">
@@ -23,5 +23,5 @@
         <origin rpy="0 0 0" xyz="0 0 0"/>
         <geometry>
-          <mesh filename="package://robotiq_hand_description/meshes/s-model_articulated/collision/link_0.STL" />
+          <mesh filename="package://iiwa_tool_description/meshes/collision/link_0.STL" />
         </geometry>
         <material name="yellow">
@@ -44,5 +44,5 @@
         <origin rpy="0 0 ${3.1416/2}" xyz="0 0.05717 0"/>
         <geometry>
-          <mesh filename="package://robotiq_hand_description/meshes/s-model_articulated/visual/link_1.STL" />
+          <mesh filename="package://iiwa_tool_description/meshes/visual/link_1.STL" />
         </geometry>
         <material name="green"/>
@@ -51,5 +51,5 @@
         <origin rpy="0 0 ${3.1416/2}" xyz="0 0.05717 0"/>
         <geometry>
-          <mesh filename="package://robotiq_hand_description/meshes/s-model_articulated/collision/link_1.STL"/>
+          <mesh filename="package://iiwa_tool_description/meshes/collision/link_1.STL"/>
         </geometry>
         <material name="yellow">
@@ -78,5 +78,5 @@
         <origin rpy="0 0 ${3.1416/2}" xyz="0 0.03810 0.0075"/>
         <geometry>
-          <mesh filename="package://robotiq_hand_description/meshes/s-model_articulated/visual/link_2.STL" />
+          <mesh filename="package://iiwa_tool_description/meshes/visual/link_2.STL" />
         </geometry>
         <material name="green"/>
@@ -85,5 +85,5 @@
         <origin rpy="0 0 ${3.1416/2}" xyz="0 0.03810 0.0075"/>
           <geometry>
-            <mesh filename="package://robotiq_hand_description/meshes/s-model_articulated/collision/link_2.STL"/>
+            <mesh filename="package://iiwa_tool_description/meshes/collision/link_2.STL"/>
           </geometry>
         <material name="yellow"/>
@@ -110,5 +110,5 @@
         <origin xyz="0 0 0" rpy="0 0 0"/>
         <geometry>
-          <mesh filename="package://robotiq_hand_description/meshes/s-model_articulated/visual/link_3.STL" />
+          <mesh filename="package://iiwa_tool_description/meshes/visual/link_3.STL" />
         </geometry>
         <material name="green"/>
@@ -117,5 +117,5 @@
         <origin xyz="0 0 0" rpy="0 0 0"/>
         <geometry>
-          <mesh filename="package://robotiq_hand_description/meshes/s-model_articulated/collision/link_3.STL"/>
+          <mesh filename="package://iiwa_tool_description/meshes/collision/link_3.STL"/>
         </geometry>
         <material name="yellow"/>
@@ -682,5 +682,5 @@
         <origin xyz="0 0 0" rpy="0 0 0"/>
         <geometry>
-          <mesh filename="package://iiwa_tool_description/meshes/visual/coupling.STL" />
+          <mesh filename="package://iiwa_tool_description/meshes//visual/coupling.STL" />
         </geometry>
         <material name="green">
@@ -691,5 +691,5 @@
         <origin rpy="0 0 0" xyz="0 0 0"/>
         <geometry>
-          <mesh filename="package://iiwa_tool_description/meshes/collision/coupling.STL" />
+          <mesh filename="package://iiwa_tool_description/meshes//collision/coupling.STL" />
         </geometry>
         <material name="yellow">
@@ -718,5 +718,5 @@
         <visual>
           <geometry>
-            <mesh filename="package://robotiq_hand_description/meshes/s-model_articulated/visual/palm.STL" />
+            <mesh filename="package://iiwa_tool_description/meshes/visual/palm.STL" />
           </geometry>
           <material name="green">
@@ -727,5 +727,5 @@
         <!-- <collision>
           <geometry>
-            <mesh filename="package://robotiq_hand_description/meshes/s-model_articulated/collision/palm.STL"/>
+            <mesh filename="package://iiwa_tool_description/meshes/collision/palm.STL"/>
           </geometry>
           <material name="yellow">

Commit message: modif 3finger xacro

File: iiwa_tool/iiwa_tool_description/urdf/iiwa14_3finger_gripper.urdf.xacro (robot description, xacro)
@@ -675,5 +675,5 @@
     <parent link="$(arg robot_name)_link_ee" />
     <child link = "coupling_link" />
-    <origin xyz="${tool_joint_offset}" rpy="0 0 0" />
+    <origin xyz="0 0 0" rpy="0 0 1" />
   </joint>
   <!-- Here we define the geometry of the coupling. the mass, center of gravity, inertial were unknown -->
@@ -707,5 +707,5 @@
     <parent link="coupling_link" />
     <child link = "palm" />
-    <origin xyz="${tool_link_offset}" rpy="0 0 0" />
+    <origin xyz="0 0 0.25" rpy="0 0 1" />
   </joint>
     <!-- Insert the fingers -->

Commit message: 3finger xacro modif

File: iiwa_tool/iiwa_tool_description/urdf/iiwa14_3finger_gripper.urdf.xacro (robot description, xacro)
@@ -707,5 +707,5 @@
     <parent link="coupling_link" />
     <child link = "palm" />
-    <origin xyz="0 0 0.25" rpy="0 0 1" />
+    <origin xyz="0 0 0" rpy="0 0 1" />
   </joint>
     <!-- Insert the fingers -->

Commit message: xacro rpy

File: iiwa_tool/iiwa_tool_description/urdf/iiwa14_3finger_gripper.urdf.xacro (robot description, xacro)
@@ -675,5 +675,5 @@
     <parent link="$(arg robot_name)_link_ee" />
     <child link = "coupling_link" />
-    <origin xyz="0 0 0" rpy="0 0 1" />
+    <origin xyz="0 0 0" rpy="0 0 0" />
   </joint>
   <!-- Here we define the geometry of the coupling. the mass, center of gravity, inertial were unknown -->
@@ -707,5 +707,5 @@
     <parent link="coupling_link" />
     <child link = "palm" />
-    <origin xyz="0 0 0" rpy="0 0 1" />
+    <origin xyz="0 0 0" rpy="0 0 ${PI / 2}" />
   </joint>
     <!-- Insert the fingers -->

Commit message: jjj

File: iiwa_tool/iiwa_tool_description/urdf/iiwa14_3finger_gripper.urdf.xacro (robot description, xacro)
@@ -675,5 +675,5 @@
     <parent link="$(arg robot_name)_link_ee" />
     <child link = "coupling_link" />
-    <origin xyz="0 0 0" rpy="0 0 0" />
+    <origin xyz="0 0 0.05" rpy="${PI / 2} ${PI / 2} ${PI / 2}" />
   </joint>
   <!-- Here we define the geometry of the coupling. the mass, center of gravity, inertial were unknown -->
@@ -707,5 +707,5 @@
     <parent link="coupling_link" />
     <child link = "palm" />
-    <origin xyz="0 0 0" rpy="0 0 ${PI / 2}" />
+    <origin xyz="0 0 0.025" rpy="0 ${PI / 2} ${PI / 2}" />
   </joint>
     <!-- Insert the fingers -->
