Commit message: test xacro

File: iiwa_tool/iiwa_tool_description/urdf/iiwa14_3finger_gripper.urdf.xacro (robot description, xacro)
@@ -675,5 +675,5 @@
     <parent link="$(arg robot_name)_link_ee" />
     <child link = "coupling_link" />
-    <origin xyz="0 0 0.05" rpy="${PI / 2} ${PI / 2} ${PI / 2}" />
+    <origin xyz="0 0 0.0" rpy="${PI / 2} ${PI / 2} ${PI / 2}" />
   </joint>
   <!-- Here we define the geometry of the coupling. the mass, center of gravity, inertial were unknown -->
@@ -707,5 +707,5 @@
     <parent link="coupling_link" />
     <child link = "palm" />
-    <origin xyz="0 0 0.025" rpy="0 ${PI / 2} ${PI / 2}" />
+    <origin xyz="0 0 0.0" rpy="0 ${PI / 2} ${PI / 2}" />
   </joint>
     <!-- Insert the fingers -->

Commit message: tetst

File: iiwa_tool/iiwa_tool_description/urdf/iiwa14_3finger_gripper.urdf.xacro (robot description, xacro)
@@ -675,5 +675,5 @@
     <parent link="$(arg robot_name)_link_ee" />
     <child link = "coupling_link" />
-    <origin xyz="0 0 0.0" rpy="${PI / 2} ${PI / 2} ${PI / 2}" />
+    <origin xyz="0 0 0.0" rpy="0 0 0" />
   </joint>
   <!-- Here we define the geometry of the coupling. the mass, center of gravity, inertial were unknown -->
@@ -707,5 +707,5 @@
     <parent link="coupling_link" />
     <child link = "palm" />
-    <origin xyz="0 0 0.0" rpy="0 ${PI / 2} ${PI / 2}" />
+    <origin xyz="0 0 0.0" rpy="0 0 0" />
   </joint>
     <!-- Insert the fingers -->

Commit message: test

File: iiwa_tool/iiwa_tool_description/urdf/iiwa14_3finger_gripper.urdf.xacro (robot description, xacro)
@@ -707,5 +707,5 @@
     <parent link="coupling_link" />
     <child link = "palm" />
-    <origin xyz="0 0 0.0" rpy="0 0 0" />
+    <origin xyz="0 0 0.0" rpy="0 ${PI/2} ${PI/2}" />
   </joint>
     <!-- Insert the fingers -->

Commit message: t

File: iiwa_tool/iiwa_tool_description/urdf/iiwa14_3finger_gripper.urdf.xacro (robot description, xacro)
@@ -675,5 +675,5 @@
     <parent link="$(arg robot_name)_link_ee" />
     <child link = "coupling_link" />
-    <origin xyz="0 0 0.0" rpy="0 0 0" />
+    <origin xyz="0 0 0.05" rpy="0 0 0" />
   </joint>
   <!-- Here we define the geometry of the coupling. the mass, center of gravity, inertial were unknown -->

Commit message: coupling rpy

File: iiwa_tool/iiwa_tool_description/urdf/iiwa14_3finger_gripper.urdf.xacro (robot description, xacro)
@@ -675,5 +675,5 @@
     <parent link="$(arg robot_name)_link_ee" />
     <child link = "coupling_link" />
-    <origin xyz="0 0 0.05" rpy="0 0 0" />
+    <origin xyz="0 0 0.05" rpy="${PI/2} 0 0" />
   </joint>
   <!-- Here we define the geometry of the coupling. the mass, center of gravity, inertial were unknown -->

Commit message: test

File: iiwa_tool/iiwa_tool_description/urdf/iiwa14_3finger_gripper.urdf.xacro (robot description, xacro)
@@ -675,5 +675,5 @@
     <parent link="$(arg robot_name)_link_ee" />
     <child link = "coupling_link" />
-    <origin xyz="0 0 0.05" rpy="${PI/2} 0 0" />
+    <origin xyz="1 2 3" rpy="${PI/2} 0 0" />
   </joint>
   <!-- Here we define the geometry of the coupling. the mass, center of gravity, inertial were unknown -->

Commit message: test

File: iiwa_tool/iiwa_tool_description/urdf/iiwa14_3finger_gripper.urdf.xacro (robot description, xacro)
@@ -675,5 +675,5 @@
     <parent link="$(arg robot_name)_link_ee" />
     <child link = "coupling_link" />
-    <origin xyz="1 2 3" rpy="${PI/2} 0 0" />
+    <origin xyz="-0.04 -0.04 0.05" rpy="${PI/2} 0 0" />
   </joint>
   <!-- Here we define the geometry of the coupling. the mass, center of gravity, inertial were unknown -->

Commit message: test

File: iiwa_tool/iiwa_tool_description/urdf/iiwa14_3finger_gripper.urdf.xacro (robot description, xacro)
@@ -675,5 +675,5 @@
     <parent link="$(arg robot_name)_link_ee" />
     <child link = "coupling_link" />
-    <origin xyz="-0.04 -0.04 0.05" rpy="${PI/2} 0 0" />
+    <origin xyz="0.0 0.0 0.0" rpy="${PI/2} 0 0" />
   </joint>
   <!-- Here we define the geometry of the coupling. the mass, center of gravity, inertial were unknown -->
@@ -707,5 +707,5 @@
     <parent link="coupling_link" />
     <child link = "palm" />
-    <origin xyz="0 0 0.0" rpy="0 ${PI/2} ${PI/2}" />
+    <origin xyz="0.0 0.0 0.0" rpy="${PI/2} ${PI/2} ${PI/2}" />
   </joint>
     <!-- Insert the fingers -->

Commit message: test

File: iiwa_tool/iiwa_tool_description/urdf/iiwa14_3finger_gripper.urdf.xacro (robot description, xacro)
@@ -707,5 +707,5 @@
     <parent link="coupling_link" />
     <child link = "palm" />
-    <origin xyz="0.0 0.0 0.0" rpy="${PI/2} ${PI/2} ${PI/2}" />
+    <origin xyz="0.0 0.0 0.05" rpy="${PI/2} ${PI/2} ${PI/2}" />
   </joint>
     <!-- Insert the fingers -->

Commit message: test

File: iiwa_tool/iiwa_tool_description/urdf/iiwa14_3finger_gripper.urdf.xacro (robot description, xacro)
@@ -707,5 +707,5 @@
     <parent link="coupling_link" />
     <child link = "palm" />
-    <origin xyz="0.0 0.0 0.05" rpy="${PI/2} ${PI/2} ${PI/2}" />
+    <origin xyz="0.05 0.1 0.0" rpy="${PI/2} ${PI/2} ${PI/2}" />
   </joint>
     <!-- Insert the fingers -->

Commit message: coupling x y

File: iiwa_tool/iiwa_tool_description/urdf/iiwa14_3finger_gripper.urdf.xacro (robot description, xacro)
@@ -675,5 +675,5 @@
     <parent link="$(arg robot_name)_link_ee" />
     <child link = "coupling_link" />
-    <origin xyz="0.0 0.0 0.0" rpy="${PI/2} 0 0" />
+    <origin xyz="0.04 0.04 0.0" rpy="${PI/2} 0 0" />
   </joint>
   <!-- Here we define the geometry of the coupling. the mass, center of gravity, inertial were unknown -->

Commit message: x y

File: iiwa_tool/iiwa_tool_description/urdf/iiwa14_3finger_gripper.urdf.xacro (robot description, xacro)
@@ -675,5 +675,5 @@
     <parent link="$(arg robot_name)_link_ee" />
     <child link = "coupling_link" />
-    <origin xyz="0.04 0.04 0.0" rpy="${PI/2} 0 0" />
+    <origin xyz="-0.04 0.04 0.0" rpy="${PI/2} 0 0" />
   </joint>
   <!-- Here we define the geometry of the coupling. the mass, center of gravity, inertial were unknown -->

Commit message: tst

File: iiwa_tool/iiwa_tool_description/urdf/iiwa14_3finger_gripper.urdf.xacro (robot description, xacro)
@@ -684,5 +684,5 @@
           <mesh filename="package://iiwa_tool_description/meshes//visual/coupling.STL" />
         </geometry>
-        <material name="green">
+        <material name="gray">
           <color rgba="0 1 0 1"/>
         </material>
@@ -693,5 +693,5 @@
           <mesh filename="package://iiwa_tool_description/meshes//collision/coupling.STL" />
         </geometry>
-        <material name="yellow">
+        <material name="gray">
           <color rgba="0 1 1 1"/>
         </material>
@@ -707,5 +707,5 @@
     <parent link="coupling_link" />
     <child link = "palm" />
-    <origin xyz="0.05 0.1 0.0" rpy="${PI/2} ${PI/2} ${PI/2}" />
+    <origin xyz="-0.05 0.1 0.0" rpy="${PI/2} ${PI/2} ${PI/2}" />
   </joint>
     <!-- Insert the fingers -->

Commit message: test

File: iiwa_tool/iiwa_tool_description/urdf/iiwa14_3finger_gripper.urdf.xacro (robot description, xacro)
@@ -707,5 +707,5 @@
     <parent link="coupling_link" />
     <child link = "palm" />
-    <origin xyz="-0.05 0.1 0.0" rpy="${PI/2} ${PI/2} ${PI/2}" />
+    <origin xyz="0.0 0.05 0.0" rpy="${PI/2} ${PI/2} ${PI/2}" />
   </joint>
     <!-- Insert the fingers -->

Commit message: ts

File: iiwa_tool/iiwa_tool_description/urdf/iiwa14_3finger_gripper.urdf.xacro (robot description, xacro)
@@ -707,5 +707,5 @@
     <parent link="coupling_link" />
     <child link = "palm" />
-    <origin xyz="0.0 0.05 0.0" rpy="${PI/2} ${PI/2} ${PI/2}" />
+    <origin xyz="0.03 0.08 0.0" rpy="${PI/2} ${PI/2} ${PI/2}" />
   </joint>
     <!-- Insert the fingers -->

Commit message: ts

File: iiwa_tool/iiwa_tool_description/urdf/iiwa14_3finger_gripper.urdf.xacro (robot description, xacro)
@@ -707,5 +707,5 @@
     <parent link="coupling_link" />
     <child link = "palm" />
-    <origin xyz="0.03 0.08 0.0" rpy="${PI/2} ${PI/2} ${PI/2}" />
+    <origin xyz="0.03 0.05 0.05" rpy="${PI/2} ${PI/2} ${PI/2}" />
   </joint>
     <!-- Insert the fingers -->

Commit message: ts

File: iiwa_tool/iiwa_tool_description/urdf/iiwa14_3finger_gripper.urdf.xacro (robot description, xacro)
@@ -707,5 +707,5 @@
     <parent link="coupling_link" />
     <child link = "palm" />
-    <origin xyz="0.03 0.05 0.05" rpy="${PI/2} ${PI/2} ${PI/2}" />
+    <origin xyz="0.03 0.05 -0.05" rpy="${PI/2} ${PI/2} ${PI/2}" />
   </joint>
     <!-- Insert the fingers -->

Commit message: ts

File: iiwa_tool/iiwa_tool_description/urdf/iiwa14_3finger_gripper.urdf.xacro (robot description, xacro)
@@ -684,6 +684,6 @@
           <mesh filename="package://iiwa_tool_description/meshes//visual/coupling.STL" />
         </geometry>
-        <material name="gray">
-          <color rgba="0 1 0 1"/>
+        <material name="Grey">
+          <!--color rgba="0 1 0 1"/-->
         </material>
       </visual>
@@ -693,6 +693,6 @@
           <mesh filename="package://iiwa_tool_description/meshes//collision/coupling.STL" />
         </geometry>
-        <material name="gray">
-          <color rgba="0 1 1 1"/>
+        <material name="Grey">
+          <!--color rgba="0 1 1 1"/-->
         </material>
       </collision>
@@ -707,5 +707,5 @@
     <parent link="coupling_link" />
     <child link = "palm" />
-    <origin xyz="0.03 0.05 -0.05" rpy="${PI/2} ${PI/2} ${PI/2}" />
+    <origin xyz="0.1 0.06 -0.05" rpy="${PI/2} ${PI/2} ${PI/2}" />
   </joint>
     <!-- Insert the fingers -->

Commit message: ts

File: iiwa_tool/iiwa_tool_description/urdf/iiwa14_3finger_gripper.urdf.xacro (robot description, xacro)
@@ -707,5 +707,5 @@
     <parent link="coupling_link" />
     <child link = "palm" />
-    <origin xyz="0.1 0.06 -0.05" rpy="${PI/2} ${PI/2} ${PI/2}" />
+    <origin xyz="-0.1 -0.1 -0.1" rpy="${PI/2} ${PI/2} ${PI/2}" />
   </joint>
     <!-- Insert the fingers -->

Commit message: ts

File: iiwa_tool/iiwa_tool_description/urdf/iiwa14_3finger_gripper.urdf.xacro (robot description, xacro)
@@ -707,5 +707,5 @@
     <parent link="coupling_link" />
     <child link = "palm" />
-    <origin xyz="-0.1 -0.1 -0.1" rpy="${PI/2} ${PI/2} ${PI/2}" />
+    <origin xyz="0.3 0.07 -0.1" rpy="${PI/2} ${PI/2} ${PI/2}" />
   </joint>
     <!-- Insert the fingers -->

Commit message: ss

File: iiwa_tool/iiwa_tool_description/urdf/iiwa14_3finger_gripper.urdf.xacro (robot description, xacro)
@@ -707,5 +707,5 @@
     <parent link="coupling_link" />
     <child link = "palm" />
-    <origin xyz="0.3 0.07 -0.1" rpy="${PI/2} ${PI/2} ${PI/2}" />
+    <origin xyz="0.1 0.1 -0.1" rpy="${PI/2} ${PI/2} ${PI/2}" />
   </joint>
     <!-- Insert the fingers -->

Commit message: ss

File: iiwa_tool/iiwa_tool_description/urdf/iiwa14_3finger_gripper.urdf.xacro (robot description, xacro)
@@ -707,5 +707,5 @@
     <parent link="coupling_link" />
     <child link = "palm" />
-    <origin xyz="0.1 0.1 -0.1" rpy="${PI/2} ${PI/2} ${PI/2}" />
+    <origin xyz="0.06 0.1 0.06" rpy="${PI/2} ${PI/2} ${PI/2}" />
   </joint>
     <!-- Insert the fingers -->

Commit message: ss

File: iiwa_tool/iiwa_tool_description/urdf/iiwa14_3finger_gripper.urdf.xacro (robot description, xacro)
@@ -707,5 +707,5 @@
     <parent link="coupling_link" />
     <child link = "palm" />
-    <origin xyz="0.06 0.1 0.06" rpy="${PI/2} ${PI/2} ${PI/2}" />
+    <origin xyz="0.06 0.08 0.04" rpy="${PI/2} ${PI/2} ${PI/2}" />
   </joint>
     <!-- Insert the fingers -->

Commit message: ss

File: iiwa_tool/iiwa_tool_description/urdf/iiwa14_3finger_gripper.urdf.xacro (robot description, xacro)
@@ -707,5 +707,5 @@
     <parent link="coupling_link" />
     <child link = "palm" />
-    <origin xyz="0.06 0.08 0.04" rpy="${PI/2} ${PI/2} ${PI/2}" />
+    <origin xyz="0.04 0.08 0.04" rpy="${PI/2} ${PI/2} ${PI/2}" />
   </joint>
     <!-- Insert the fingers -->

Commit message: black

File: iiwa_tool/iiwa_tool_description/urdf/iiwa14_3finger_gripper.urdf.xacro (robot description, xacro)
@@ -16,6 +16,6 @@
           <mesh filename="package://iiwa_tool_description/meshes/visual/link_0.STL" />
         </geometry>
-        <material name="green">
-          <color rgba="0 0 0 0.5"/>
+        <material name="Black">
+          <color rgba="0 1 0 1"/>
         </material>
       </visual>
@@ -26,5 +26,5 @@
         </geometry>
         <material name="yellow">
-          <color rgba="0 0 0 0.5"/>
+          <color rgba="0 1 1 1"/>
         </material>
       </collision>
@@ -46,5 +46,5 @@
           <mesh filename="package://iiwa_tool_description/meshes/visual/link_1.STL" />
         </geometry>
-        <material name="green"/>
+        <material name="Black"/>
       </visual>
       <collision>
@@ -54,5 +54,5 @@
         </geometry>
         <material name="yellow">
-          <color rgba="0 0 0 0.5"/>
+          <color rgba="0 1 1 1"/>
         </material>
       </collision>
@@ -80,5 +80,5 @@
           <mesh filename="package://iiwa_tool_description/meshes/visual/link_2.STL" />
         </geometry>
-        <material name="green"/>
+        <material name="Black"/>
       </visual>
       <collision>
@@ -112,5 +112,5 @@
           <mesh filename="package://iiwa_tool_description/meshes/visual/link_3.STL" />
         </geometry>
-        <material name="green"/>
+        <material name="Black"/>
       </visual>
       <collision>
@@ -685,5 +685,5 @@
         </geometry>
         <material name="Grey">
-          <!--color rgba="0 0 0 0.5"/-->
+          <!--color rgba="0 1 0 1"/-->
         </material>
       </visual>
@@ -694,5 +694,5 @@
         </geometry>
         <material name="Grey">
-          <!--color rgba="0 0 0 0.5"/-->
+          <!--color rgba="0 1 1 1"/-->
         </material>
       </collision>
@@ -720,6 +720,6 @@
             <mesh filename="package://iiwa_tool_description/meshes/visual/palm.STL" />
           </geometry>
-          <material name="green">
-            <color rgba="0 0 0 0.5"/>
+          <material name="Black">
+            <color rgba="0 1 0 1"/>
           </material>
         </visual>
@@ -730,5 +730,5 @@
           </geometry>
           <material name="yellow">
-            <color rgba="0 0 0 0.5"/>
+            <color rgba="0 1 1 1"/>
           </material>
         </collision> -->
@@ -740,5 +740,5 @@
           </geometry>
           <material name="yellow">
-            <color rgba="0 0 0 0.5"/>
+            <color rgba="0 1 1 1"/>
           </material>
         </collision>

Commit message: 0.7

File: iiwa_tool/iiwa_tool_description/urdf/iiwa14_3finger_gripper.urdf.xacro (robot description, xacro)
@@ -707,5 +707,5 @@
     <parent link="coupling_link" />
     <child link = "palm" />
-    <origin xyz="0.04 0.08 0.04" rpy="${PI/2} ${PI/2} ${PI/2}" />
+    <origin xyz="0.04 0.07 0.04" rpy="${PI/2} ${PI/2} ${PI/2}" />
   </joint>
     <!-- Insert the fingers -->

Commit message: grey

File: iiwa_tool/iiwa_tool_description/urdf/iiwa14_3finger_gripper.urdf.xacro (robot description, xacro)
@@ -16,5 +16,5 @@
           <mesh filename="package://iiwa_tool_description/meshes/visual/link_0.STL" />
         </geometry>
-        <material name="Black">
+        <material name="Grey">
           <color rgba="0 1 0 1"/>
         </material>
@@ -46,5 +46,5 @@
           <mesh filename="package://iiwa_tool_description/meshes/visual/link_1.STL" />
         </geometry>
-        <material name="Black"/>
+        <material name="Grey"/>
       </visual>
       <collision>
@@ -80,5 +80,5 @@
           <mesh filename="package://iiwa_tool_description/meshes/visual/link_2.STL" />
         </geometry>
-        <material name="Black"/>
+        <material name="Grey"/>
       </visual>
       <collision>
@@ -112,5 +112,5 @@
           <mesh filename="package://iiwa_tool_description/meshes/visual/link_3.STL" />
         </geometry>
-        <material name="Black"/>
+        <material name="Grey"/>
       </visual>
       <collision>
@@ -720,5 +720,5 @@
             <mesh filename="package://iiwa_tool_description/meshes/visual/palm.STL" />
           </geometry>
-          <material name="Black">
+          <material name="Grey">
             <color rgba="0 1 0 1"/>
           </material>

Commit message: gold

File: iiwa_tool/iiwa_tool_description/urdf/iiwa14_3finger_gripper.urdf.xacro (robot description, xacro)
@@ -25,5 +25,5 @@
           <mesh filename="package://iiwa_tool_description/meshes/collision/link_0.STL" />
         </geometry>
-        <material name="yellow">
+        <material name="Gold">
           <color rgba="0 1 1 1"/>
         </material>
@@ -53,5 +53,5 @@
           <mesh filename="package://iiwa_tool_description/meshes/collision/link_1.STL"/>
         </geometry>
-        <material name="yellow">
+        <material name="Gold">
           <color rgba="0 1 1 1"/>
         </material>
@@ -87,5 +87,5 @@
             <mesh filename="package://iiwa_tool_description/meshes/collision/link_2.STL"/>
           </geometry>
-        <material name="yellow"/>
+        <material name="Gold"/>
       </collision>
       <inertial>
@@ -119,5 +119,5 @@
           <mesh filename="package://iiwa_tool_description/meshes/collision/link_3.STL"/>
         </geometry>
-        <material name="yellow"/>
+        <material name="Gold"/>
       </collision>
       <inertial>
@@ -729,5 +729,5 @@
             <mesh filename="package://iiwa_tool_description/meshes/collision/palm.STL"/>
           </geometry>
-          <material name="yellow">
+          <material name="Gold">
             <color rgba="0 1 1 1"/>
           </material>
@@ -739,5 +739,5 @@
             <box size="0.1 0.1 0.1"/>
           </geometry>
-          <material name="yellow">
+          <material name="Gold">
             <color rgba="0 1 1 1"/>
           </material>

Commit message: orange

File: iiwa_tool/iiwa_tool_description/urdf/iiwa14_3finger_gripper.urdf.xacro (robot description, xacro)
@@ -25,5 +25,5 @@
           <mesh filename="package://iiwa_tool_description/meshes/collision/link_0.STL" />
         </geometry>
-        <material name="Gold">
+        <material name="Orange">
           <color rgba="0 1 1 1"/>
         </material>
@@ -53,5 +53,5 @@
           <mesh filename="package://iiwa_tool_description/meshes/collision/link_1.STL"/>
         </geometry>
-        <material name="Gold">
+        <material name="Orange">
           <color rgba="0 1 1 1"/>
         </material>
@@ -87,5 +87,5 @@
             <mesh filename="package://iiwa_tool_description/meshes/collision/link_2.STL"/>
           </geometry>
-        <material name="Gold"/>
+        <material name="Orange"/>
       </collision>
       <inertial>
@@ -119,5 +119,5 @@
           <mesh filename="package://iiwa_tool_description/meshes/collision/link_3.STL"/>
         </geometry>
-        <material name="Gold"/>
+        <material name="Orange"/>
       </collision>
       <inertial>
@@ -729,5 +729,5 @@
             <mesh filename="package://iiwa_tool_description/meshes/collision/palm.STL"/>
           </geometry>
-          <material name="Gold">
+          <material name="Orange">
             <color rgba="0 1 1 1"/>
           </material>
@@ -739,5 +739,5 @@
             <box size="0.1 0.1 0.1"/>
           </geometry>
-          <material name="Gold">
+          <material name="Orange">
             <color rgba="0 1 1 1"/>
           </material>

Commit message: grey

File: iiwa_tool/iiwa_tool_description/urdf/iiwa14_3finger_gripper.urdf.xacro (robot description, xacro)
@@ -25,5 +25,5 @@
           <mesh filename="package://iiwa_tool_description/meshes/collision/link_0.STL" />
         </geometry>
-        <material name="Orange">
+        <material name="Grey">
           <color rgba="0 1 1 1"/>
         </material>
@@ -53,5 +53,5 @@
           <mesh filename="package://iiwa_tool_description/meshes/collision/link_1.STL"/>
         </geometry>
-        <material name="Orange">
+        <material name="Grey">
           <color rgba="0 1 1 1"/>
         </material>
@@ -87,5 +87,5 @@
             <mesh filename="package://iiwa_tool_description/meshes/collision/link_2.STL"/>
           </geometry>
-        <material name="Orange"/>
+        <material name="Grey"/>
       </collision>
       <inertial>
@@ -119,5 +119,5 @@
           <mesh filename="package://iiwa_tool_description/meshes/collision/link_3.STL"/>
         </geometry>
-        <material name="Orange"/>
+        <material name="Grey"/>
       </collision>
       <inertial>
@@ -729,5 +729,5 @@
             <mesh filename="package://iiwa_tool_description/meshes/collision/palm.STL"/>
           </geometry>
-          <material name="Orange">
+          <material name="Grey">
             <color rgba="0 1 1 1"/>
           </material>
@@ -739,5 +739,5 @@
             <box size="0.1 0.1 0.1"/>
           </geometry>
-          <material name="Orange">
+          <material name="Grey">
             <color rgba="0 1 1 1"/>
           </material>

Commit message: color

File: iiwa_tool/iiwa_tool_description/urdf/iiwa14_3finger_gripper.urdf.xacro (robot description, xacro)
@@ -651,4 +651,6 @@
 	<box size="0.60 0.60 0.76"/>
       </geometry>
+      <material name="Grey">
+      </material>
     </visual>
     <collision>
@@ -657,4 +659,6 @@
 	<box size="0.60 0.60 0.76"/>
       </geometry>
+      <material name="Grey">
+      </material>
     </collision>
   </link>
