Commit message: aaa

File: iiwa_3finger_description/urdf/iiwa_3finger.urdf (robot description, URDF)
Before this commit: robot iiwa_3finger, 51 links, 50 joints
Links:
- link coupling_link: geometry collision mesh filename=package://iiwa_3finger_description/meshes/collision/couplin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; visual mesh filename=package://iiwa_3finger_description/meshes/visual/coupling.S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
- link finger_1_link_0: geometry collision mesh filename=package://iiwa_3finger_description/meshes/collision/link_0.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; visual mesh filename=package://iiwa_3finger_description/meshes/visual/link_0.STL
- link finger_1_link_1: geometry collision mesh filename=package://iiwa_3finger_description/meshes/collision/link_1.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; visual mesh filename=package://iiwa_3finger_description/meshes/visual/link_1.STL
- link finger_1_link_2: geometry collision mesh filename=package://iiwa_3finger_description/meshes/collision/link_2.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; visual mesh filename=package://iiwa_3finger_description/meshes/visual/link_2.STL
- link finger_1_link_3: geometry collision mesh filename=package://iiwa_3finger_description/meshes/collision/link_3.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; visual mesh filename=package://iiwa_3finger_description/meshes/visual/link_3.STL
- link finger_2_link_0: geometry collision mesh filename=package://iiwa_3finger_description/meshes/collision/link_0.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; visual mesh filename=package://iiwa_3finger_description/meshes/visual/link_0.STL
- link finger_2_link_1: geometry collision mesh filename=package://iiwa_3finger_description/meshes/collision/link_1.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; visual mesh filename=package://iiwa_3finger_description/meshes/visual/link_1.STL
- link finger_2_link_2: geometry collision mesh filename=package://iiwa_3finger_description/meshes/collision/link_2.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; visual mesh filename=package://iiwa_3finger_description/meshes/visual/link_2.STL
- link finger_2_link_3: geometry collision mesh filename=package://iiwa_3finger_description/meshes/collision/link_3.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; visual mesh filename=package://iiwa_3finger_description/meshes/visual/link_3.STL
- link finger_middle_link_0: geometry collision mesh filename=package://iiwa_3finger_description/meshes/collision/link_0.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; visual mesh filename=package://iiwa_3finger_description/meshes/visual/link_0.STL
- link finger_middle_link_1: geometry collision mesh filename=package://iiwa_3finger_description/meshes/collision/link_1.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; visual mesh filename=package://iiwa_3finger_description/meshes/visual/link_1.STL
- link finger_middle_link_2: geometry collision mesh filename=package://iiwa_3finger_description/meshes/collision/link_2.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; visual mesh filename=package://iiwa_3finger_description/meshes/visual/link_2.STL
- link finger_middle_link_3: geometry collision mesh filename=package://iiwa_3finger_description/meshes/collision/link_3.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; visual mesh filename=package://iiwa_3finger_description/meshes/visual/link_3.STL
- link palm: geometry collision box size=0.1 0.1 0.1; collision mesh filename=package://iiwa_3finger_description/meshes/collision/palm.STL

File: iiwa_3finger_description/urdf/iiwa_3finger.urdf.xacro (robot description, xacro)
@@ -1,7 +1,5 @@
 <?xml version="1.0"?>
 <!-- Here we define the robot, we named it "iiwa14_3finger_gripper" -->
-<robot xmlns:xacro="http://www.ros.org/wiki/xacro" name="iiwa_3finger">
-  <!-- Import Rviz colors -->
-  <xacro:include filename="$(find iiwa_description)/urdf/materials.xacro" />
+<robot name="iiwa_3finger" xmlns:xacro="http://www.ros.org/wiki/xacro">
   <!--Import the iiwa14 macro -->
   <xacro:include filename="$(find iiwa_description)/urdf/iiwa14.xacro"/>
@@ -16,5 +14,4 @@
   If you don't want to have that you can define a basic world link (see commented lines)
   -->
-  <xacro:macro name="iiwa_3finger" params="parent hardware_interface robot_name *origin">
     <!--     <link name="world"/> -->
   <link name="world">
@@ -68,5 +65,5 @@
         <origin rpy="0 0 0" xyz="0 0 0"/>
         <geometry>
-          <mesh filename="package://iiwa_3finger_description/meshes/visual/collision/coupling.STL" />
+          <mesh filename="package://iiwa_3finger_description/meshes/collision/coupling.STL" />
         </geometry>
         <material name="Grey">
@@ -95,19 +92,19 @@
         <visual>
           <geometry>
-            <mesh filename="package://iiwa_tool_description/meshes/visual/palm.STL" />
+            <mesh filename="package://iiwa_3finger_description/meshes/visual/palm.STL" />
           </geometry>
-          <material name="Green">
+          <material name="Black">
             <!-- <color rgba="0 1 0 1"/> -->
           </material>
         </visual>
         <!-- Mesh collision -->
-        <!-- <collision>
+        <collision>
           <geometry>
-            <mesh filename="package://iiwa_tool_description/meshes/collision/palm.STL"/>
+            <mesh filename="package://iiwa_3finger_description/meshes/collision/palm.STL"/>
           </geometry>
           <material name="Grey">
             <color rgba="0 1 1 1"/>
           </material>
-        </collision> -->
+        </collision>
         <!-- Simple shape collision -->
         <collision>
@@ -170,4 +167,3 @@
       <implicitSpringDamper>1</implicitSpringDamper>
     </gazebo>
-    </xacro:macro>
 </robot>

File: iiwa_3finger_description/urdf/robotiq_finger.urdf.xacro (robot description, xacro)
@@ -4,6 +4,4 @@
   <!-- Import Rviz colors -->
   <xacro:include filename="$(find iiwa_description)/urdf/materials.xacro" />
-  <!--Import the iiwa14 macro -->
-  <xacro:include filename="$(find iiwa_description)/urdf/iiwa14.xacro"/>
   <!--Build finger model -->
   <xacro:macro name="robotiq_finger" params="prefix">
@@ -23,5 +21,5 @@
         <origin rpy="0 0 0" xyz="0 0 0"/>
         <geometry>
-          <mesh filename="package://iiwa_tool_description/meshes/collision/link_0.STL" />
+          <mesh filename="package://iiwa_3finger_description/meshes/collision/link_0.STL" />
         </geometry>
         <material name="Grey">
@@ -44,5 +42,5 @@
         <origin rpy="0 0 ${3.1416/2}" xyz="0 0.05717 0"/>
         <geometry>
-          <mesh filename="package://iiwa_tool_description/meshes/visual/link_1.STL" />
+          <mesh filename="package://iiwa_3finger_description/meshes/visual/link_1.STL" />
         </geometry>
         <material name="Grey"/>
@@ -51,5 +49,5 @@
         <origin rpy="0 0 ${3.1416/2}" xyz="0 0.05717 0"/>
         <geometry>
-          <mesh filename="package://iiwa_tool_description/meshes/collision/link_1.STL"/>
+          <mesh filename="package://iiwa_3finger_description/meshes/collision/link_1.STL"/>
         </geometry>
         <material name="Grey">
@@ -78,5 +76,5 @@
         <origin rpy="0 0 ${3.1416/2}" xyz="0 0.03810 0.0075"/>
         <geometry>
-          <mesh filename="package://iiwa_tool_description/meshes/visual/link_2.STL" />
+          <mesh filename="package://iiwa_3finger_description/meshes/visual/link_2.STL" />
         </geometry>
         <material name="Grey"/>
@@ -85,5 +83,5 @@
         <origin rpy="0 0 ${3.1416/2}" xyz="0 0.03810 0.0075"/>
           <geometry>
-            <mesh filename="package://iiwa_tool_description/meshes/collision/link_2.STL"/>
+            <mesh filename="package://iiwa_3finger_description/meshes/collision/link_2.STL"/>
           </geometry>
         <material name="Grey"/>
@@ -110,5 +108,5 @@
         <origin xyz="0 0 0" rpy="0 0 0"/>
         <geometry>
-          <mesh filename="package://iiwa_tool_description/meshes/visual/link_3.STL" />
+          <mesh filename="package://iiwa_3finger_description/meshes/visual/link_3.STL" />
         </geometry>
         <material name="Grey"/>
@@ -117,5 +115,5 @@
         <origin xyz="0 0 0" rpy="0 0 0"/>
         <geometry>
-          <mesh filename="package://iiwa_tool_description/meshes/collision/link_3.STL"/>
+          <mesh filename="package://iiwa_3finger_description/meshes/collision/link_3.STL"/>
         </geometry>
         <material name="Grey"/>
